Commit message: Controladores com Erro

File: urdf/chiquinho.xacro (robot description, xacro)
@@ -25,5 +25,5 @@
               size="0.075 0.065 0.455"
               color="White"/>
-    <robot_joint parent="link_1" child="link_2" type="prismatic"
+    <!-- <robot_joint parent="link_1" child="link_2" type="prismatic"
              origin_xyz="0 -0.2275 0" origin_rpy="0 0 0"
              axis="0 0 1"
@@ -48,4 +48,9 @@
       izz="0.00008333"
       size="0.1 0.1 0.1"
-      color="Red"/>
+      color="Red"/> -->
+    <!-- END Robot description -->
+    <!-- BNG Gazebo -->
+      <gazebo>
+            <plugin name="gazebo_ros_control" filename="libgazebo_ros_control.so"/>
+      </gazebo>
 </robot>

File: urdf/link_joint.xacro (robot description, xacro)
@@ -18,4 +18,14 @@
             <child link="${child}" />
         </joint>
+        <transmission name="trans_${parent}__${child}">
+            <type>transmission_interface/SimpleTransmission</type>
+            <joint name="${parent}__${child}">
+                <hardwareInterface>hardware_interface/EffortJointInterface</hardwareInterface>
+            </joint>
+            <actuator name="motor_${parent}__${child}">
+                <hardwareInterface>hardware_interface/EffortJointInterface</hardwareInterface>
+                <mechanicalReduction>1</mechanicalReduction>
+            </actuator>
+        </transmission>
     </xacro:macro>
     <xacro:macro name="box_link" params="name origin_xyz origin_rpy mass ixx ixy ixz iyy iyz izz size color">
